File: hardware/can-hat.kicad_pcb (KiCad board)
At the start: 0 parts

Commit message: feat: finish pcb
Parts:
- added C1: 100nF, Capacitor_SMD:C_0201_0603Metric, F.Cu at (58.0, 51.5)
- added C10: 100nF, Capacitor_SMD:C_0201_0603Metric, F.Cu at (95.5, 58.5)
- added C11: 100nF, Capacitor_SMD:C_0201_0603Metric, F.Cu at (91.7, 67.0)
- added C12: 100nF, Capacitor_SMD:C_0201_0603Metric, F.Cu at (86.5, 67.0)
- added C13: 10µF, Capacitor_SMD:C_0805_2012Metric, F.Cu at (55.5, 45.5)
- added C14: 10µF, Capacitor_SMD:C_0805_2012Metric, F.Cu at (51.0, 45.5)
- added C2: 100nF, Capacitor_SMD:C_0201_0603Metric, F.Cu at (58.7, 64.0)
- added C3: 100nF, Capacitor_SMD:C_0201_0603Metric, F.Cu at (49.0, 70.5)
- added C4: 100nF, Capacitor_SMD:C_0201_0603Metric, F.Cu at (54.7, 70.5)
- added C5: 100nF, Capacitor_SMD:C_0201_0603Metric, F.Cu at (76.2, 50.0)
- added C6: 100nF, Capacitor_SMD:C_0201_0603Metric, F.Cu at (73.0, 70.0)
- added C7: 100nF, Capacitor_SMD:C_0201_0603Metric, F.Cu at (77.3, 62.0)
- added C8: 100nF, Capacitor_SMD:C_0201_0603Metric, F.Cu at (67.5, 70.0)
- added C9: 100nF, Capacitor_SMD:C_0201_0603Metric, F.Cu at (94.5, 46.5)
- added G***: LOGO, LOGO, F.Cu at (103.8, 56.0)
- added G***: LOGO, LOGO, F.Cu at (46.0, 49.2)
- added G***: LOGO, LOGO, F.Cu at (46.5, 82.5)
- added J1: RPi_GPIO, RPI_Hat:RPI_Hat_B+, F.Cu at (73.8, 40.5)
- added J2: CAN0, Degson:SHDRRA2W80P0X350_1X2_780X920X722P, F.Cu at (57.8, 84.5)
- added J3: CAN1, Degson:SHDRRA2W80P0X350_1X2_780X920X722P, F.Cu at (67.8, 84.5)
- added J4: CAN2, Degson:SHDRRA2W80P0X350_1X2_780X920X722P, F.Cu at (77.8, 84.5)
- added R1: 10kΩ, Resistor_SMD:R_0201_0603Metric, F.Cu at (54.5, 63.5)
- added R2: 120Ω, Resistor_SMD:R_0201_0603Metric, F.Cu at (56.2, 72.0)
- added R3: 120Ω, Resistor_SMD:R_0201_0603Metric, F.Cu at (75.0, 71.5)
- added R4: 10kΩ, Resistor_SMD:R_0201_0603Metric, F.Cu at (72.8, 62.0)
- added R5: 120Ω, Resistor_SMD:R_0201_0603Metric, F.Cu at (93.7, 66.0)
- added R6: 10kΩ, Resistor_SMD:R_0201_0603Metric, F.Cu at (91.7, 59.0)
- added R7: 1kΩ, Resistor_SMD:R_0201_0603Metric, F.Cu at (100.0, 72.0)
- added R8: 3.9kΩ, Resistor_SMD:R_0201_0603Metric, F.Cu at (98.0, 72.0)
- added R9: 3.9kΩ, Resistor_SMD:R_0201_0603Metric, F.Cu at (96.0, 72.0)
- added REF**: OSHW-Logo2_7.3x6mm_SilkScreen, Symbol:OSHW-Logo2_7.3x6mm_SilkScreen, F.Cu at (101.5, 47.8)
- added TP1: WriteProtect Enable, TestPoint:TestPoint_2Pads_Pitch2.54mm_Drill0.8mm, F.Cu at (99.2, 80.5)
- added U1: MCP2518FD-xQBB, PCM_JLCPCB:SOIC-14_L8.7-W3.9-P1.27-LS6.0-BL, F.Cu at (55.5, 57.0)
- added U2: MCP2562FD-E/SN, Package_SO:SOIC-8_3.9x4.9mm_P1.27mm, F.Cu at (52.0, 67.0)
- added U3: MCP2518FD-xQBB, PCM_JLCPCB:SOIC-14_L8.7-W3.9-P1.27-LS6.0-BL, F.Cu at (73.5, 55.5)
- added U4: MCP2562FD-E/SN, Package_SO:SOIC-8_3.9x4.9mm_P1.27mm, F.Cu at (70.5, 65.5)
- added U5: MCP2518FD-xQBB, PCM_JLCPCB:SOIC-14_L8.7-W3.9-P1.27-LS6.0-BL, F.Cu at (92.0, 52.5)
- added U6: MCP2562FD-E/SN, Package_SO:SOIC-8_3.9x4.9mm_P1.27mm, F.Cu at (89.0, 62.5)
- added U7: AT24C32, Package_SO:SOIC-8_3.9x4.9mm_P1.27mm, F.Cu at (98.0, 75.5)
- added Y1: 40MHZ Oscillator, Crystal:Crystal_SMD_5032-4Pin_5.0x3.2mm, F.Cu at (60.6, 67.0)
- added Y2: 40MHZ Oscillator, Crystal:Crystal_SMD_5032-4Pin_5.0x3.2mm, F.Cu at (79.0, 65.0)
- added Y3: 40MHZ Oscillator, Crystal:Crystal_SMD_5032-4Pin_5.0x3.2mm, F.Cu at (97.5, 62.0)
Routing:
- net +3.3V: track 0.00 -> 202.3 mm, vias 0 -> 9
- net +5V: track 0.00 -> 135.3 mm, vias 0 -> 3
- net GND: track 0.00 -> 102.2 mm, vias 0 -> 15
- net /SPI1_SCLK: track 0.00 -> 55.7 mm, vias 0 -> 2
- net /SPI1_MOSI: track 0.00 -> 54.7 mm, vias 0 -> 2
- net /SPI3_CE0: track 0.00 -> 49.6 mm, vias 0 -> 3
- net /SPI1_MISO: track 0.00 -> 48.0 mm, vias 0 -> 2
- net /SPI3_MOSI: track 0.00 -> 46.3 mm
- net /ID_SC: track 0.00 -> 44.7 mm, vias 0 -> 1
- net /ID_SD: track 0.00 -> 43.6 mm, vias 0 -> 1
- net /SPI3_MISO: track 0.00 -> 41.5 mm
- net /SPI3_SCLK: track 0.00 -> 40.8 mm
- net /CAN2/CAN_P: track 0.00 -> 35.9 mm
- net /CAN2/CAN_N: track 0.00 -> 34.6 mm
- net /SPI1_CE1: track 0.00 -> 30.5 mm
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- added copper zone on B.Cu, net GND
Other:
- board outline added: 65 x 56.5 mm
- copper layers 0 -> 2
- board text added: "(Short to GND)"
- board text added: "1317"
- board text added: "CAN0"
- board text added: "CAN1"
- board text added: "CAN2"
- board text added: "U1"
- board text added: "U3"
- board text added: "U5"
- board text added: "U7"
- board text added: "Write Enable"
- board text added: "^^"
- board text added: "a dunkirk corp design"
- board text added: "made for"
