File: hardware/can-hat.kicad_sch (KiCad schematic)
At the start: 0 parts

Commit message: feat: add can channels
Other:
- added sheet CAN0 (can_channel.kicad_sch)
- added sheet CAN1 (can_channel.kicad_sch)
- added sheet CAN2 (can_channel.kicad_sch)

Commit message: feat: finish the schematic
Parts:
- added C13, C14: 10µF, Capacitor_SMD:C_0805_2012Metric, symbol Device:C
- added J1: RPi_GPIO, RPI_Hat:RPI_Hat_B+, symbol RPi_Hat:RPi_GPIO
- added J2: CAN0, Degson:SHDRRA2W80P0X350_1X2_780X920X722P, symbol Connector_Generic:Conn_01x02
- added J3: CAN1, Degson:SHDRRA2W80P0X350_1X2_780X920X722P, symbol Connector_Generic:Conn_01x02
- added J4: CAN2, Degson:SHDRRA2W80P0X350_1X2_780X920X722P, symbol Connector_Generic:Conn_01x02
- added R7: 1kΩ, Resistor_SMD:R_0201_0603Metric, symbol Device:R_Small
- added R8, R9: 3.9kΩ, Resistor_SMD:R_0201_0603Metric, symbol Device:R_Small
- added TP1: WP TestPoint, TestPoint:TestPoint_Pad_1.5x1.5mm, symbol Connector:TestPoint
- added U7: AT24C32, Package_SO:SOIC-8_3.9x4.9mm_P1.27mm, symbol Memory_EEPROM:24C02Cx-x-SN
Connections:
- net SPI1_MISO: now also J1.35 (BCM19_MISO_PCM_FS)
- net SPI1_MOSI: now also J1.38 (BCM20_MOSI_PCM_DI)
- net SPI1_SCLK: now also J1.40 (BCM21_SCLK_PCM_DO)
- net SPI3_MISO: now also J1.26 (BCM7_CE1)
- net SPI3_MOSI: now also J1.31 (BCM6)
- net SPI3_SCLK: now also J1.29 (BCM5)
- new net +3.3V: C13.1, J1.1 (3.3V), J1.17 (3.3V), R7.1, R8.2, R9.2, U7.8 (VCC)
- new net +5V: C14.1, J1.2 (5V), J1.4 (5V)
- new net CAN0/CAN_N: J2.2 (Pin_2)
- new net CAN0/CAN_P: J2.1 (Pin_1)
- new net CAN1/CAN_N: J3.2 (Pin_2)
- new net CAN1/CAN_P: J3.1 (Pin_1)
- new net CAN2/CAN_N: J4.2 (Pin_2)
- new net CAN2/CAN_P: J4.1 (Pin_1)
- new net GND: C13.2, C14.2, J1.14 (GND), J1.20 (GND), J1.25 (GND), J1.30 (GND), J1.34 (GND), J1.39 (GND), J1.6 (GND), J1.9 (GND), U7.1 (A0), U7.2 (A1), U7.3 (A2), U7.4 (GND)
- new net ID_SC: J1.28 (BCM1_ID_SC), R8.1, U7.6 (SCL)
- new net ID_SD: J1.27 (BCM0_ID_SD), R9.1, U7.5 (SDA)
- new net SPI1_CE0: J1.12 (BCM18_PCM_C)
- new net SPI1_CE1: J1.11 (BCM17)
- new net SPI1_INT0: J1.16 (BCM23)
- new net SPI1_INT1: J1.18 (BCM24)
- new net SPI3_CE0: J1.7 (BCM4_GPCLK0)
- new net SPI3_INT0: J1.15 (BCM22)
- new net WriteProtect: R7.2, TP1.1, U7.7 (WP)
- no-connect marks 0 -> 14
Other:
- sheet CAN0 ports: added CAN_N, CAN_P; removed CANH, CANL
- sheet CAN1 ports: added CAN_N, CAN_P; removed CANH, CANL
- sheet CAN2 ports: added CAN_N, CAN_P; removed CANH, CANL
- company: (none) -> Kieran Klukas
- title: (none) -> CAN Hat

Commit message: feat: finish pcb
Parts:
- removed TP1: WP TestPoint, TestPoint:TestPoint_Pad_1.5x1.5mm, symbol Connector:TestPoint
- added TP1: WriteProtect Enable, TestPoint:TestPoint_2Pads_Pitch2.54mm_Drill0.8mm, symbol Connector:TestPoint_2Pole
Connections:
- net GND: now also TP1.2
- net WriteProtect: now also TP1.1
Other:
- moved on the sheet: R7
Changed lines of the file:
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@@
 	)
 	(junction
-		(at 86.36 67.31)
+		(at 85.09 63.5)
 		(diameter 0)
 		(color 0 0 0 0)
@@
 	(wire
 		(pts
-			(xy 86.36 67.31) (xy 86.36 69.85)
+			(xy 85.09 63.5) (xy 85.09 71.12)
 		)
 		(stroke
@@
 	(wire
 		(pts
+			(xy 85.09 71.12) (xy 88.9 71.12)
+		)
+		(stroke
+			(width 0)
+			(type default)
+		)
+	)
+	(wire
+		(pts
 			(xy 91.44 30.48) (xy 91.44 33.02)
 		)
@@
 	(wire
 		(pts
-			(xy 88.9 67.31) (xy 86.36 67.31)
+			(xy 87.63 63.5) (xy 85.09 63.5)
 		)
 		(stroke
@@
 	(wire
 		(pts
+			(xy 99.06 71.12) (xy 101.6 71.12)
+		)
+		(stroke
+			(width 0)
+			(type default)
+		)
+	)
+	(wire
+		(pts
 			(xy 175.26 59.69) (xy 172.72 59.69)
 		)
@@
 	(wire
 		(pts
-			(xy 86.36 59.69) (xy 86.36 67.31)
+			(xy 85.09 58.42) (xy 85.09 63.5)
 		)
 		(stroke
@@
 	(wire
 		(pts
-			(xy 93.98 67.31) (xy 99.06 67.31)
+			(xy 92.71 63.5) (xy 100.33 63.5)
 		)
 		(stroke
@@
 	(wire
 		(pts
-			(xy 99.06 67.31) (xy 99.06 66.04)
-		)
-		(stroke
-			(width 0)
-			(type default)
-		)
-	)
-	(wire
-		(pts
 			(xy 124.46 54.61) (xy 111.76 54.61)
 		)
@@
 	)
 	(label "WriteProtect"
-		(at 86.36 59.69 0)
+		(at 85.09 58.42 0)
 		(effects
 			(font
@@
 	(symbol
 		(lib_id "Device:R_Small")
-		(at 91.44 67.31 270)
+		(at 90.17 63.5 270)
 		(unit 1)
 		(exclude_from_sim no)
@@
 		(on_board yes)
 		(dnp no)
-		(fields_autoplaced yes)
 		(property "Reference" "R7"
-			(at 91.44 62.23 90)
+			(at 90.17 59.944 90)
 			(effects
 				(font
@@
 		)
 		(property "Value" "1kΩ"
-			(at 91.44 64.77 90)
+			(at 90.17 61.468 90)
 			(effects
 				(font
@@
 		)
 		(property "Footprint" "Resistor_SMD:R_0201_0603Metric"
-			(at 91.44 67.31 0)
+			(at 90.17 63.5 0)
 			(effects
 				(font
@@
 		)
 		(property "Datasheet" "~"
-			(at 91.44 67.31 0)
+			(at 90.17 63.5 0)
 			(effects
 				(font
@@
 		)
 		(property "Description" "Resistor, small symbol"
-			(at 91.44 67.31 0)
+			(at 90.17 63.5 0)
 			(effects
 				(font
@@
 	(symbol
 		(lib_id "power:+3.3V")
-		(at 99.06 66.04 0)
+		(at 100.33 63.5 0)
 		(unit 1)
 		(exclude_from_sim no)
@@
 		(fields_autoplaced yes)
 		(property "Reference" "#PWR043"
-			(at 99.06 69.85 0)
+			(at 100.33 67.31 0)
 			(effects
 				(font
@@
 		)
 		(property "Value" "+3.3V"
-			(at 99.06 60.96 0)
+			(at 100.33 58.42 0)
 			(effects
 				(font
@@
 		)
 		(property "Footprint" ""
-			(at 99.06 66.04 0)
+			(at 100.33 63.5 0)
 			(effects
 				(font
@@
 		)
 		(property "Datasheet" ""
-			(at 99.06 66.04 0)
+			(at 100.33 63.5 0)
 			(effects
 				(font
@@
 		)
 		(property "Description" "Power symbol creates a global label with name \"+3.3V\""
-			(at 99.06 66.04 0)
+			(at 100.33 63.5 0)
 			(effects
 				(font
@@
 	(symbol
 		(lib_id "power:GND")
+		(at 101.6 71.12 0)
+		(unit 1)
+		(exclude_from_sim no)
+		(in_bom yes)
+		(on_board yes)
+		(dnp no)
+		(fields_autoplaced yes)
+		(property "Reference" "#PWR055"
+			(at 101.6 77.47 0)
+			(effects
+				(font
+					(size 1.27 1.27)
+				)
+				(hide yes)
+			)
+		)
+		(property "Value" "GND"
+			(at 101.6 76.2 0)
+			(effects
+				(font
+					(size 1.27 1.27)
+				)
+			)
+		)
+		(property "Footprint" ""
+			(at 101.6 71.12 0)
+			(effects
+				(font
+					(size 1.27 1.27)
+				)
+				(hide yes)
+			)
+		)
+		(property "Datasheet" ""
+			(at 101.6 71.12 0)
+			(effects
+				(font
+					(size 1.27 1.27)
+				)
+				(hide yes)
+			)
+		)
+		(property "Description" "Power symbol creates a global label with name \"GND\" , ground"
+			(at 101.6 71.12 0)
+			(effects
+				(font
+					(size 1.27 1.27)
+				)
+				(hide yes)
+			)
+		)
+		(pin "1"
+		)
+		(instances
+			(project "can-hat"
+				(path "/bfdea6a0-b5c8-4489-9fa0-a972c3ff35f2"
+					(reference "#PWR055")
+					(unit 1)
+				)
+			)
+		)
+	)
+	(symbol
+		(lib_id "power:GND")
 		(at 185.42 39.37 0)
 		(unit 1)
@@
 	)
 	(symbol
-		(lib_id "Connector:TestPoint")
-		(at 86.36 69.85 180)
+		(lib_id "Connector:TestPoint_2Pole")
+		(at 93.98 71.12 0)
 		(unit 1)
 		(exclude_from_sim no)
@@
 		(on_board yes)
 		(dnp no)
-		(fields_autoplaced yes)
 		(property "Reference" "TP1"
-			(at 88.9 71.8819 0)
+			(at 94.488 66.04 0)
 			(effects
 				(font
 					(size 1.27 1.27)
 				)
-				(justify right)
 			)
 		)
-		(property "Value" "WP TestPoint"
-			(at 88.9 74.4219 0)
+		(property "Value" "WriteProtect Enable"
+			(at 94.742 68.072 0)
 			(effects
 				(font
 					(size 1.27 1.27)
 				)
-				(justify right)
 			)
 		)
-		(property "Footprint" "TestPoint:TestPoint_Pad_1.5x1.5mm"
-			(at 81.28 69.85 0)
+		(property "Footprint" "TestPoint:TestPoint_2Pads_Pitch2.54mm_Drill0.8mm"
+			(at 93.98 71.12 0)
 			(effects
 				(font
@@
 		)
 		(property "Datasheet" "~"
-			(at 81.28 69.85 0)
+			(at 93.98 71.12 0)
 			(effects
 				(font
@@
 			)
 		)
-		(property "Description" "test point"
-			(at 86.36 69.85 0)
+		(property "Description" "2-polar test point"
+			(at 93.98 71.12 0)
 			(effects
 				(font
@@
 		(pin "1"
 		)
+		(pin "2"
+		)
 		(instances

Commit message: chore: add parts and fix bom
Parts:
- C13, C14: LCSC (none) -> C15850
- J1, TP1: now left out of the parts list
- J2, J3, J4: LCSC (none) -> C5632692
- R7: LCSC (none) -> C21190
- R8, R9: LCSC (none) -> C23196
- U7: LCSC (none) -> C60583
Changed lines of the file:
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@@
+			)
+		)
+		(property "LCSC" "C5632692"
+			(at 0 0 0)
+			(effects
+				(font
+					(size 1.27 1.27)
+				)
+				(hide yes)
 			)
 		)
@@
 			)
 		)
+		(property "LCSC" "C15850"
+			(at 0 0 0)
+			(effects
+				(font
+					(size 1.27 1.27)
+				)
+				(hide yes)
+			)
+		)
 		(pin "2"
 		)
@@
 		(property "Description" "2-Kbit (256 x 8-bit) I2C Serial EEPROM, chip address inputs (A0, A1, A2), write-protect pin (WP), 4.5..5.5V supply, SOIC-8"
 			(at 68.58 35.56 0)
+			(effects
+				(font
+					(size 1.27 1.27)
+				)
+				(hide yes)
+			)
+		)
+		(property "LCSC" "C60583"
+			(at 0 0 0)
 			(effects
 				(font
@@
 			)
 		)
+		(property "LCSC" "C21190"
+			(at 0 0 0)
+			(effects
+				(font
+					(size 1.27 1.27)
+				)
+				(hide yes)
+			)
+		)
 		(pin "2"
 		)
@@
 			)
 		)
+		(property "LCSC" "C23196"
+			(at 0 0 0)
+			(effects
+				(font
+					(size 1.27 1.27)
+				)
+				(hide yes)
+			)
+		)
 		(pin "2"
 		)
@@
 			)
 		)
+		(property "LCSC" "C5632692"
+			(at 0 0 0)
+			(effects
+				(font
+					(size 1.27 1.27)
+				)
+				(hide yes)
+			)
+		)
 		(pin "1"
 		)
@@
 		(property "Description" "Resistor, small symbol"
 			(at 81.28 27.94 0)
+			(effects
+				(font
+					(size 1.27 1.27)
+				)
+				(hide yes)
+			)
+		)
+		(property "LCSC" "C23196"
+			(at 0 0 0)
 			(effects
 				(font
@@
 			)
 		)
+		(property "LCSC" "C5632692"
+			(at 0 0 0)
+			(effects
+				(font
+					(size 1.27 1.27)
+				)
+				(hide yes)
+			)
+		)
 		(pin "1"
 		)
@@
 			)
 		)
+		(property "LCSC" "C15850"
+			(at 0 0 0)
+			(effects
+				(font
+					(size 1.27 1.27)
+				)
+				(hide yes)
+			)
+		)
 		(pin "2"
 		)
@@
 		(unit 1)
 		(exclude_from_sim no)
-		(in_bom yes)
+		(in_bom no)
 		(on_board yes)
 		(dnp no)
@@
 		(unit 1)
 		(exclude_from_sim no)
-		(in_bom yes)
-		(on_board yes)
-		(dnp no)
+		(in_bom no)
+		(on_board yes)
+		(dnp no)
