File: hardware/can_channel.kicad_sch (KiCad schematic)
At the start: 9 parts, among them U1 MCP2518FD-xQBB, U2 MCP2562FD-E/SN, Y1 40MHZ Oscillator

Commit message: feat: finish the schematic
Parts:
- removed C2: 100nF, symbol Device:C_Small
- added C?: 100nF, Capacitor_SMD:C_0201_0603Metric, symbol Device:C_Small
- C?: renamed from C1; footprint (none) -> Capacitor_SMD:C_0201_0603Metric
- C?: renamed from C3; footprint (none) -> Capacitor_SMD:C_0201_0603Metric
- C?: renamed from C4; footprint (none) -> Capacitor_SMD:C_0201_0603Metric
- R?: renamed from R1; footprint (none) -> Resistor_SMD:R_0201_0603Metric
- R?: renamed from R2; footprint (none) -> Resistor_SMD:R_0201_0603Metric
- Y?: renamed from Y1; footprint Oscillator:Oscillator_SMD_Abracon_ASCO-4Pin_1.6x1.2mm -> Crystal:Crystal_SMD_5032-4Pin_5.0x3.2mm
- renumbered U1 to U?, U2 to U?
Connections:
- net +3.3V: now also Y?.1 (Tri-State), C?.1; no longer Y?.3 (OUT)
- net GND: now also C?.2
- net XO_OUT: now also Y?.3 (OUT); no longer Y?.1 (Tri-State)
- net CANH renamed CAN_P
- net CANL renamed CAN_N
- net RXCAN renamed XCAN_N
- net XCAN_N: now also U?.1 (TXCAN); no longer U?.2 (RXCAN)
- net TXCAN renamed XCAN_P
- net XCAN_P: now also U?.2 (RXCAN); no longer U?.1 (TXCAN)
Other:
- moved on the sheet: C?, R?, U?, Y?

Commit message: feat: finish pcb
Parts:
- gave numbers to parts that had none: 9
Changed lines of the file:
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@@
 		(dnp no)
 		(fields_autoplaced yes)
-		(property "Reference" "#PWR?"
+		(property "Reference" "#PWR06"
 			(at 72.39 38.1 0)
 			(effects
@@
 		(dnp no)
 		(fields_autoplaced yes)
-		(property "Reference" "#PWR?"
+		(property "Reference" "#PWR03"
 			(at 72.39 26.67 0)
 			(effects
@@
 		(on_board yes)
 		(dnp no)
-		(property "Reference" "Y?"
+		(property "Reference" "Y1"
 			(at 101.092 22.352 0)
 			(effects
@@
 		(dnp no)
 		(fields_autoplaced yes)
-		(property "Reference" "#PWR?"
+		(property "Reference" "#PWR011"
 			(at 116.84 54.61 0)
 			(effects
@@
 		(dnp no)
 		(fields_autoplaced yes)
-		(property "Reference" "R?"
+		(property "Reference" "R1"
 			(at 130.81 59.6899 0)
 			(effects
@@
 		(dnp no)
 		(fields_autoplaced yes)
-		(property "Reference" "#PWR?"
+		(property "Reference" "#PWR012"
 			(at 128.27 71.12 0)
 			(effects
@@
 		(dnp no)
 		(fields_autoplaced yes)
-		(property "Reference" "#PWR?"
+		(property "Reference" "#PWR04"
 			(at 91.44 46.99 0)
 			(effects
@@
 		(dnp no)
 		(fields_autoplaced yes)
-		(property "Reference" "#PWR?"
+		(property "Reference" "#PWR010"
 			(at 116.84 66.04 0)
 			(effects
@@
 		(dnp no)
 		(fields_autoplaced yes)
-		(property "Reference" "U?"
+		(property "Reference" "U1"
 			(at 42.7833 35.56 0)
 			(effects
@@
 		(dnp no)
 		(fields_autoplaced yes)
-		(property "Reference" "#PWR?"
+		(property "Reference" "#PWR05"
 			(at 29.21 39.37 0)
 			(effects
@@
 		(dnp no)
 		(fields_autoplaced yes)
-		(property "Reference" "C?"
+		(property "Reference" "C2"
 			(at 74.93 26.6762 0)
 			(effects
@@
 		(dnp no)
 		(fields_autoplaced yes)
-		(property "Reference" "#PWR?"
+		(property "Reference" "#PWR01"
 			(at 40.64 27.94 0)
 			(effects
@@
 		(dnp no)
 		(fields_autoplaced yes)
-		(property "Reference" "R?"
+		(property "Reference" "R2"
 			(at 96.52 57.15 90)
 			(effects
@@
 		(dnp no)
 		(fields_autoplaced yes)
-		(property "Reference" "C?"
+		(property "Reference" "C1"
 			(at 31.75 27.9462 0)
 			(effects
@@
 		(dnp no)
 		(fields_autoplaced yes)
-		(property "Reference" "U?"
+		(property "Reference" "U2"
 			(at 143.1133 36.83 0)
 			(effects
@@
 		(dnp no)
 		(fields_autoplaced yes)
-		(property "Reference" "#PWR?"
+		(property "Reference" "#PWR07"
 			(at 129.54 40.64 0)
 			(effects
@@
 		(dnp no)
 		(fields_autoplaced yes)
-		(property "Reference" "#PWR?"
+		(property "Reference" "#PWR02"
 			(at 40.64 71.12 0)
 			(effects
@@
 		(dnp no)
 		(fields_autoplaced yes)
-		(property "Reference" "C?"
+		(property "Reference" "C3"
 			(at 132.08 29.2162 0)
 			(effects
@@
 		(dnp no)
 		(fields_autoplaced yes)
-		(property "Reference" "#PWR?"
+		(property "Reference" "#PWR09"
 			(at 140.97 67.31 0)
 			(effects
@@
 		(dnp no)
 		(fields_autoplaced yes)
-		(property "Reference" "#PWR?"
+		(property "Reference" "#PWR08"
 			(at 140.97 29.21 0)
 			(effects
@@
 		(dnp no)
 		(fields_autoplaced yes)
-		(property "Reference" "C?"
+		(property "Reference" "C4"
 			(at 119.38 54.6162 0)
 			(effects

Commit message: chore: add parts and fix bom
Parts:
- C1, C2, C3, C4: LCSC (none) -> C14663
- R1: LCSC (none) -> C25803
- R2: LCSC (none) -> C25879
- U1: LCSC (none) -> C626759
- U2: LCSC (none) -> C511335
- Y1: LCSC (none) -> C295515
Changed lines of the file:
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@@
+			)
+		)
+		(property "LCSC" "C295515"
+			(at 0 0 0)
+			(effects
+				(font
+					(size 1.27 1.27)
+				)
+				(hide yes)
 			)
 		)
@@
 			)
 		)
+		(property "LCSC" "C25803"
+			(at 0 0 0)
+			(effects
+				(font
+					(size 1.27 1.27)
+				)
+				(hide yes)
+			)
+		)
 		(pin "1"
 		)
@@
 			)
 		)
+		(property "LCSC" "C626759"
+			(at 0 0 0)
+			(effects
+				(font
+					(size 1.27 1.27)
+				)
+				(hide yes)
+			)
+		)
 		(pin "8"
 		)
@@
 			)
 		)
+		(property "LCSC" "C14663"
+			(at 0 0 0)
+			(effects
+				(font
+					(size 1.27 1.27)
+				)
+				(hide yes)
+			)
+		)
 		(pin "2"
 		)
@@
 			)
 		)
+		(property "LCSC" "C25879"
+			(at 0 0 0)
+			(effects
+				(font
+					(size 1.27 1.27)
+				)
+				(hide yes)
+			)
+		)
 		(pin "1"
 		)
@@
 			)
 		)
+		(property "LCSC" "C14663"
+			(at 0 0 0)
+			(effects
+				(font
+					(size 1.27 1.27)
+				)
+				(hide yes)
+			)
+		)
 		(pin "2"
 		)
@@
 			)
 		)
+		(property "LCSC" "C511335"
+			(at 0 0 0)
+			(effects
+				(font
+					(size 1.27 1.27)
+				)
+				(hide yes)
+			)
+		)
 		(pin "4"
 		)
@@
 			)
 		)
+		(property "LCSC" "C14663"
+			(at 0 0 0)
+			(effects
+				(font
+					(size 1.27 1.27)
+				)
+				(hide yes)
+			)
+		)
 		(pin "2"
 		)
@@
 			(effects
 				(font
+					(size 1.27 1.27)
+				)
+				(hide yes)
+			)
+		)
+		(property "LCSC" "C14663"
+			(at 0 0 0)
+			(effects
+				(font
