File: hardware/CANopy_branch.kicad_sch (KiCad schematic)
At the start: 9 parts, among them U1 MCP2518FD-xQBB, U2 MCP2562FD-E/SN, Y1 40MHZ Oscillator

Commit message: feat: rename to CANopy
Other:
- title: CAN Channel -> CANopy Branch
Changed lines of the file:
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@@
 	(paper "User" 177.8 120.65)
 	(title_block
-		(title "CAN Channel")
+		(title "CANopy Branch")
 		(date "2026-04-25")
 		(rev "1")
@@
 		)
 		(instances
-			(project "can_channel"
+			(project "CANopy_branch"
 				(path "/9116dce4-ee6f-4c1d-b606-42cf2e075a74"
 					(reference "#PWR?")
@@
 				)
 			)
-			(project "can-hat"
+			(project "CANopy"
 				(path "/bfdea6a0-b5c8-4489-9fa0-a972c3ff35f2/00e2c20b-7be4-4f83-a3f0-21fb1d83928e"
 					(reference "#PWR0101")
@@
 		)
 		(instances
-			(project "can_channel"
+			(project "CANopy_branch"
 				(path "/9116dce4-ee6f-4c1d-b606-42cf2e075a74"
 					(reference "#PWR?")
@@
 				)
 			)
-			(project "can-hat"
+			(project "CANopy"
 				(path "/bfdea6a0-b5c8-4489-9fa0-a972c3ff35f2/00e2c20b-7be4-4f83-a3f0-21fb1d83928e"
 					(reference "#PWR0102")
@@
 		)
 		(instances
-			(project "can_channel"
+			(project "CANopy_branch"
 				(path "/9116dce4-ee6f-4c1d-b606-42cf2e075a74"
 					(reference "Y?")
@@
 				)
 			)
-			(project "can-hat"
+			(project "CANopy"
 				(path "/bfdea6a0-b5c8-4489-9fa0-a972c3ff35f2/00e2c20b-7be4-4f83-a3f0-21fb1d83928e"
 					(reference "Y2")
@@
 		)
 		(instances
-			(project "can_channel"
+			(project "CANopy_branch"
 				(path "/9116dce4-ee6f-4c1d-b606-42cf2e075a74"
 					(reference "#PWR?")
@@
 				)
 			)
-			(project "can-hat"
+			(project "CANopy"
 				(path "/bfdea6a0-b5c8-4489-9fa0-a972c3ff35f2/00e2c20b-7be4-4f83-a3f0-21fb1d83928e"
 					(reference "#PWR019")
@@
 		)
 		(instances
-			(project "can_channel"
+			(project "CANopy_branch"
 				(path "/9116dce4-ee6f-4c1d-b606-42cf2e075a74"
 					(reference "R?")
@@
 				)
 			)
-			(project "can-hat"
+			(project "CANopy"
 				(path "/bfdea6a0-b5c8-4489-9fa0-a972c3ff35f2/00e2c20b-7be4-4f83-a3f0-21fb1d83928e"
 					(reference "R4")
@@
 		)
 		(instances
-			(project "can_channel"
+			(project "CANopy_branch"
 				(path "/9116dce4-ee6f-4c1d-b606-42cf2e075a74"
 					(reference "#PWR?")
@@
 				)
 			)
-			(project "can-hat"
+			(project "CANopy"
 				(path "/bfdea6a0-b5c8-4489-9fa0-a972c3ff35f2/00e2c20b-7be4-4f83-a3f0-21fb1d83928e"
 					(reference "#PWR021")
@@
 		)
 		(instances
-			(project "can_channel"
+			(project "CANopy_branch"
 				(path "/9116dce4-ee6f-4c1d-b606-42cf2e075a74"
 					(reference "#PWR?")
@@
 				)
 			)
-			(project "can-hat"
+			(project "CANopy"
 				(path "/bfdea6a0-b5c8-4489-9fa0-a972c3ff35f2/00e2c20b-7be4-4f83-a3f0-21fb1d83928e"
 					(reference "#PWR017")
@@
 		)
 		(instances
-			(project "can_channel"
+			(project "CANopy_branch"
 				(path "/9116dce4-ee6f-4c1d-b606-42cf2e075a74"
 					(reference "#PWR?")
@@
 				)
 			)
-			(project "can-hat"
+			(project "CANopy"
 				(path "/bfdea6a0-b5c8-4489-9fa0-a972c3ff35f2/00e2c20b-7be4-4f83-a3f0-21fb1d83928e"
 					(reference "#PWR020")
@@
 		)
 		(instances
-			(project "can_channel"
+			(project "CANopy_branch"
 				(path "/9116dce4-ee6f-4c1d-b606-42cf2e075a74"
 					(reference "U?")
@@
 				)
 			)
-			(project "can-hat"
+			(project "CANopy"
 				(path "/bfdea6a0-b5c8-4489-9fa0-a972c3ff35f2/00e2c20b-7be4-4f83-a3f0-21fb1d83928e"
 					(reference "U3")
@@
 		)
 		(instances
-			(project "can_channel"
+			(project "CANopy_branch"
 				(path "/9116dce4-ee6f-4c1d-b606-42cf2e075a74"
 					(reference "#PWR?")
@@
 				)
 			)
-			(project "can-hat"
+			(project "CANopy"
 				(path "/bfdea6a0-b5c8-4489-9fa0-a972c3ff35f2/00e2c20b-7be4-4f83-a3f0-21fb1d83928e"
 					(reference "#PWR013")
@@
 		)
 		(instances
-			(project "can_channel"
+			(project "CANopy_branch"
 				(path "/9116dce4-ee6f-4c1d-b606-42cf2e075a74"
 					(reference "C?")
@@
 				)
 			)
-			(project "can-hat"
+			(project "CANopy"
 				(path "/bfdea6a0-b5c8-4489-9fa0-a972c3ff35f2/00e2c20b-7be4-4f83-a3f0-21fb1d83928e"
 					(reference "C6")
@@
 		)
 		(instances
-			(project "can_channel"
+			(project "CANopy_branch"
 				(path "/9116dce4-ee6f-4c1d-b606-42cf2e075a74"
 					(reference "#PWR?")
@@
 				)
 			)
-			(project "can-hat"
+			(project "CANopy"
 				(path "/bfdea6a0-b5c8-4489-9fa0-a972c3ff35f2/00e2c20b-7be4-4f83-a3f0-21fb1d83928e"
 					(reference "#PWR014")
@@
 		)
 		(instances
-			(project "can_channel"
+			(project "CANopy_branch"
 				(path "/9116dce4-ee6f-4c1d-b606-42cf2e075a74"
 					(reference "R?")
@@
 				)
 			)
-			(project "can-hat"
+			(project "CANopy"
 				(path "/bfdea6a0-b5c8-4489-9fa0-a972c3ff35f2/00e2c20b-7be4-4f83-a3f0-21fb1d83928e"
 					(reference "R3")
@@
 		)
 		(instances
-			(project "can_channel"
+			(project "CANopy_branch"
 				(path "/9116dce4-ee6f-4c1d-b606-42cf2e075a74"
 					(reference "C?")
@@
 				)
 			)
-			(project "can-hat"
+			(project "CANopy"
 				(path "/bfdea6a0-b5c8-4489-9fa0-a972c3ff35f2/00e2c20b-7be4-4f83-a3f0-21fb1d83928e"
 					(reference "C5")
@@
 		)
 		(instances
-			(project "can_channel"
+			(project "CANopy_branch"
 				(path "/9116dce4-ee6f-4c1d-b606-42cf2e075a74"
 					(reference "U?")
@@
 				)
 			)
-			(project "can-hat"
+			(project "CANopy"
 				(path "/bfdea6a0-b5c8-4489-9fa0-a972c3ff35f2/00e2c20b-7be4-4f83-a3f0-21fb1d83928e"
 					(reference "U4")
@@
 		)
 		(instances
-			(project "can_channel"
+			(project "CANopy_branch"
 				(path "/9116dce4-ee6f-4c1d-b606-42cf2e075a74"
 					(reference "#PWR?")
@@
 				)
 			)
-			(project "can-hat"
+			(project "CANopy"
 				(path "/bfdea6a0-b5c8-4489-9fa0-a972c3ff35f2/00e2c20b-7be4-4f83-a3f0-21fb1d83928e"
 					(reference "#PWR022")
@@
 		)
 		(instances
-			(project "can_channel"
+			(project "CANopy_branch"
 				(path "/9116dce4-ee6f-4c1d-b606-42cf2e075a74"
 					(reference "#PWR?")
@@
 				)
 			)
-			(project "can-hat"
+			(project "CANopy"
 				(path "/bfdea6a0-b5c8-4489-9fa0-a972c3ff35f2/00e2c20b-7be4-4f83-a3f0-21fb1d83928e"
 					(reference "#PWR015")
@@
 		)
 		(instances
-			(project "can_channel"
+			(project "CANopy_branch"
 				(path "/9116dce4-ee6f-4c1d-b606-42cf2e075a74"
 					(reference "C?")
@@
 				)
 			)
-			(project "can-hat"
+			(project "CANopy"
 				(path "/bfdea6a0-b5c8-4489-9fa0-a972c3ff35f2/00e2c20b-7be4-4f83-a3f0-21fb1d83928e"
 					(reference "C8")
@@
 		)
 		(instances
-			(project "can_channel"
+			(project "CANopy_branch"
 				(path "/9116dce4-ee6f-4c1d-b606-42cf2e075a74"
 					(reference "#PWR?")
@@
 				)
 			)
-			(project "can-hat"
+			(project "CANopy"
 				(path "/bfdea6a0-b5c8-4489-9fa0-a972c3ff35f2/00e2c20b-7be4-4f83-a3f0-21fb1d83928e"
 					(reference "#PWR024")
@@
 		)
 		(instances
-			(project "can_channel"
+			(project "CANopy_branch"
 				(path "/9116dce4-ee6f-4c1d-b606-42cf2e075a74"
 					(reference "#PWR?")
@@
 				)
 			)
-			(project "can-hat"
+			(project "CANopy"
 				(path "/bfdea6a0-b5c8-4489-9fa0-a972c3ff35f2/00e2c20b-7be4-4f83-a3f0-21fb1d83928e"
 					(reference "#PWR023")
@@
 		)
 		(instances
-			(project "can_channel"
+			(project "CANopy_branch"
 				(path "/9116dce4-ee6f-4c1d-b606-42cf2e075a74"
 					(reference "C?")
@@
 				)
 			)
-			(project "can-hat"
+			(project "CANopy"
 				(path "/bfdea6a0-b5c8-4489-9fa0-a972c3ff35f2/00e2c20b-7be4-4f83-a3f0-21fb1d83928e"
 					(reference "C7")

Commit message: feat: update schematic with proper cap sizes
Parts:
- C1, C2, C3, C4: value 100nF -> 1µF; footprint Capacitor_SMD:C_0201_0603Metric -> Capacitor_SMD:C_0603_1608Metric
- R1, R2: footprint Resistor_SMD:R_0201_0603Metric -> Resistor_SMD:R_0603_1608Metric
Changed lines of the file:
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@@
 			)
 		)
-		(property "Footprint" "Resistor_SMD:R_0201_0603Metric"
+		(property "Footprint" "Resistor_SMD:R_0603_1608Metric"
 			(at 128.27 60.96 0)
 			(effects
@@
 			)
 		)
-		(property "Value" "100nF"
+		(property "Value" "1µF"
 			(at 74.93 29.2162 0)
 			(effects
@@
 			)
 		)
-		(property "Footprint" "Capacitor_SMD:C_0201_0603Metric"
+		(property "Footprint" "Capacitor_SMD:C_0603_1608Metric"
 			(at 72.39 27.94 0)
 			(effects
@@
 			)
 		)
-		(property "Footprint" "Resistor_SMD:R_0201_0603Metric"
+		(property "Footprint" "Resistor_SMD:R_0603_1608Metric"
 			(at 96.52 61.722 90)
 			(effects
@@
 			)
 		)
-		(property "Value" "100nF"
+		(property "Value" "1µF"
 			(at 31.75 30.4862 0)
 			(effects
@@
 			)
 		)
-		(property "Footprint" "Capacitor_SMD:C_0201_0603Metric"
+		(property "Footprint" "Capacitor_SMD:C_0603_1608Metric"
 			(at 29.21 29.21 0)
 			(effects
@@
 			)
 		)
-		(property "Value" "100nF"
+		(property "Value" "1µF"
 			(at 132.08 31.7562 0)
 			(effects
@@
 			)
 		)
-		(property "Footprint" "Capacitor_SMD:C_0201_0603Metric"
+		(property "Footprint" "Capacitor_SMD:C_0603_1608Metric"
 			(at 129.54 30.48 0)
 			(effects
@@
 			)
 		)
-		(property "Value" "100nF"
+		(property "Value" "1µF"
 			(at 119.38 57.1562 0)
 			(effects
@@
 			)
 		)
-		(property "Footprint" "Capacitor_SMD:C_0201_0603Metric"
+		(property "Footprint" "Capacitor_SMD:C_0603_1608Metric"
 			(at 116.84 55.88 0)
 			(effects

Commit message: feat: first pass reroute
Parts:
- added TP2: CAN INTER RX TX, symbol Connector:TestPoint_Alt
- renumbered C2 to C6, Y1 to Y2
Connections:
- net GND: no longer Y2.2 (GND)
- net XCAN_N: no longer names the net of U1.1 (TXCAN), U2.4 (RXD)
- net XCAN_N: now also TP2.1 (TX)
- net XCAN_P: no longer names the net of U1.2 (RXCAN), U2.1 (TXD)
- net XCAN_P: now also TP2.1 (TX)
- net XO_OUT: no longer names the net of U1.6 (OSC1), Y2.3 (OUT)
Other:
- moved on the sheet: C1, C3, C4, C6, R1, R2, U1, U2, Y2
